File: LPC2148_stick.sch (KiCad schematic (older format))
At the start: 72 parts, among them CON1 BARREL_JACK, CON2 USB-MINI-B, IC1 LM1117, IC2 LM1117, P1 CONN_01X40, P2 JTAG, P3 CONN_01X40, P4 USB Operation Selection, Q1 BC856, SW1 RST, SW2 Power, SW3 ISP, SW4 ISP, SW5 User Sw1, U1 LPC2148, X1 3.768KHz, X2 12MHz

Commit message: added final designs
Connections:
- net at P1.16 (P16): now also U1.2 (AD1.7/CAP0.0/MAT0.0/P0.22); no longer U1.1 (PWM5/AD1.6/CAP1.3/P0.21)
- net PO.22: no longer names the net of P1.17 (P17)
- net PO.22: now also U1.1 (PWM5/AD1.6/CAP1.3/P0.21); no longer U1.2 (AD1.7/CAP0.0/MAT0.0/P0.22)
Changed lines of the file:
@@
 	1    0    0    -1
 $EndComp
-Text Label 2490 4560 2    59   ~ 0
-PO.22
-Text Label 1220 4460 0    39   ~ 0
-PO.22
 Text Label 2490 5460 2    39   ~ 0
 CONNECT
@@
 	1220 4360 2490 4360
 Wire Wire Line
-	1860 4460 2490 4460
-Wire Wire Line
-	1860 4460 1860 4560
-Wire Wire Line
-	1860 4560 1220 4560
-Wire Wire Line
 	1220 4660 2180 4660
 Wire Wire Line
@@
 Wire Wire Line
 	2280 6620 2280 7120
+Wire Wire Line
+	2490 4460 1220 4460
+Wire Wire Line
+	2490 4560 1220 4560
 $EndSCHEMATC
