File: LPC2148_stick.kicad_pcb (KiCad board)
At the start: 2 copper layers, 132 x 51 mm, 72 parts, among them CON1 BARREL_JACK, CON2 USB-MINI-B, IC1 LM1117, IC2 LM1117, P1 CONN_01X40, P2 JTAG, P3 CONN_01X40, P4 USB Operation Selection, Q1 BC856, SW1 RST, SW2 Power, SW3 ISP, SW4 ISP, SW5 User Sw1, U1 LPC2148, X1 3.768KHz, X2 12MHz

Commit message: added final designs
Parts:
- added EE_LOGO: , logo:EE_LOGO(2), B.Cu at (168.0, 59.6)
- D6: footprint Diodes_SMD:Diode-SMA_Handsoldering -> EE:ZenerDiode_SMD
- R13, R14, R15, R16: moved to F.Cu
- moved R13 32.6 mm to (126.4, 52.8)
- moved D2 31.5 mm to (125.9, 49.0), turned to 315 degrees
- moved R14 30.3 mm to (123.8, 52.8)
- moved D3 29.3 mm to (123.3, 49.0), turned to 315 degrees
- moved R15 28.8 mm to (121.3, 52.8)
- moved R16 28.1 mm to (118.7, 52.8)
- moved D4 27.8 mm to (120.8, 49.0), turned to 315 degrees
- moved D5 27.3 mm to (118.2, 49.0), turned to 315 degrees
- moved C10 7.39 mm to (132.5, 62.2)
- moved C3 5.66 mm to (132.5, 54.2)
- moved L1 5.57 mm to (133.6, 51.3)
- moved C4 5.57 mm to (132.5, 56.0)
- moved L2 5.48 mm to (131.4, 51.3)
- moved L3 5.39 mm to (132.2, 57.8)
- moved C6 5.28 mm to (118.0, 79.6), turned to 45 degrees
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Connections:
- P1 pad 17: /PO.22 -> Net-(P1-Pad17)
- U1 pad 1: Net-(P1-Pad16) -> Net-(P1-Pad17)
- U1 pad 2: /PO.22 -> Net-(P1-Pad16)
Routing:
- net GND: track 0.00 -> 658.7 mm, vias 0 -> 18
- net +3.3VP: track 0.00 -> 453.1 mm, vias 0 -> 12
- net +5V: track 0.00 -> 204.3 mm, vias 0 -> 3
- net /TMS: track 0.00 -> 160.7 mm, vias 0 -> 4
- net /VBUS: track 0.00 -> 155.6 mm, vias 0 -> 3
- net /TDI: track 0.00 -> 149.8 mm, vias 0 -> 1
- net /TXD1: track 0.00 -> 149.6 mm, vias 0 -> 1
- net /CONNECT: track 0.00 -> 149.2 mm, vias 0 -> 2
- net /RXD1: track 0.00 -> 137.3 mm, vias 0 -> 3
- net HOST_USB_D+: track 0.00 -> 132.2 mm, vias 0 -> 1
- net /SSEL1: track 0.00 -> 126.0 mm, vias 0 -> 2
- net /RXD0: track 0.00 -> 120.3 mm, vias 0 -> 2
- net HOST_USB_D-: track 0.00 -> 119.0 mm, vias 0 -> 1
- net /~TRST: track 0.00 -> 117.2 mm, vias 0 -> 3
- net /TCK: track 0.00 -> 113.3 mm, vias 0 -> 4
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- added copper zone on F.Cu, net +3.3VP
- added copper zone on B.Cu, net GND
Other:
- net class Default: clearance 0.254 -> 0.1778
- rule trace_clearance: 0.254 -> 0.1778
- board text added: "+3V3"
- board text added: "+5V"
- board text added: "B-Mask"
- board text added: "COMP"
- board text added: "ExploreEmbedded.com"
- board text added: "F-Mask"
- board text added: "GND"
- board text added: "MISO1"
- board text added: "MOSI1"
- board text added: "NC"
- board text added: "P0.00"
- board text added: "P0.01"
- board text added: "P0.02"
- board text added: "P0.03"
- board text added: "P0.04"
- board text added: "P0.05"
- board text added: "P0.06"
- board text added: "P0.07"
- board text added: "P0.08"
- board text added: "P0.09"
- board text added: "P0.10"
- board text added: "P0.11"
- board text added: "P0.12"
- board text added: "P0.13"
- board text added: "P0.16"
- board text added: "P0.17"
- board text added: "P0.18"
- board text added: "P0.19"
- board text added: "P0.20"
- board text added: "P0.21"
- board text added: "P0.22"
- board text added: "P0.23"
- board text added: "P0.25"
- board text added: "P0.28"
- board text added: "P0.29"
- board text added: "P0.30"
- board text added: "P0.31"
- board text added: "P1.16"
- board text added: "P1.17"
- board text added: "P1.18"
- board text added: "P1.19"
- board text added: "P1.20"
- board text added: "P1.21"
- board text added: "P1.22"
- board text added: "P1.23"
- board text added: "P1.24"
- board text added: "P1.25"
- board text added: "P1.26"
- board text added: "P1.27"
- board text added: "P1.28"
- board text added: "P1.29"
- board text added: "P1.30"
- board text added: "P1.31"
- board text added: "PRI_BLD"
- board text added: "RXD0"
- board text added: "RXD1"
- board text added: "SCK1"
- board text added: "SCL"
- board text added: "SDA"
- board text added: "SOLD"
- board text added: "SSEL1"
- board text added: "TXD0"
- board text added: "TXD1"
- board text added: "USB+"
- board text added: "USB-"
- board text added: "~RST"

Commit message: CORRECTED FILES
Other:
- board text added: "BLD_D+"
- board text added: "BLD_D-"
- board text added: "HOST_D+"
- board text added: "HOST_D-"
- board text added: "USB"
Changed lines of the file:
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@@
     (links 231)
     (no_connects 0)
-    (area 41.224287 19.150001 219 92.084402)
+    (area 58.924999 40.924999 196.552323 92.084402)
     (thickness 1.6)
-    (drawings 95)
+    (drawings 97)
     (tracks 2021)
     (zones 0)
@@
     (descr "Crystal, Quarz, Rundgehaeuse, round, horizontal, liegend, Uhrenquarz, Diam. 2mm,")
     (tags "Crystal, Quarz, Rundgehaeuse, round, horizontal, liegend, Uhrenquarz, Diam. 2mm,")
-    (fp_text reference X1 (at 1.778 5.588 180) (layer B.SilkS)
+    (fp_text reference X1 (at 0.154 6.88 180) (layer B.SilkS)
       (effects (font (size 0.6 0.6) (thickness 0.15)) (justify mirror))
     )
@@
     (tags "capacitor 0603")
     (attr smd)
-    (fp_text reference C1 (at 0 1.9 90) (layer B.SilkS)
-      (effects (font (size 1 1) (thickness 0.15)) (justify mirror))
+    (fp_text reference C1 (at 2.074 0.56 180) (layer B.SilkS)
+      (effects (font (size 0.6 0.6) (thickness 0.15)) (justify mirror))
     )
-    (fp_text value 22pf (at 0 -1.9 90) (layer B.Fab)
+    (fp_text value 22pf (at 0 -1.9 90) (layer B.Fab) hide
       (effects (font (size 1 1) (thickness 0.15)) (justify mirror))
     )
@@
     (tags "capacitor 0603")
     (attr smd)
-    (fp_text reference C2 (at 0 1.9 90) (layer B.SilkS)
-      (effects (font (size 1 1) (thickness 0.15)) (justify mirror))
+    (fp_text reference C2 (at 2.324 0.132 180) (layer B.SilkS)
+      (effects (font (size 0.6 0.6) (thickness 0.15)) (justify mirror))
     )
-    (fp_text value 22pf (at 0 -1.9 90) (layer B.Fab)
+    (fp_text value 22pf (at 0 -1.9 90) (layer B.Fab) hide
       (effects (font (size 1 1) (thickness 0.15)) (justify mirror))
     )
@@
       (effects (font (size 0.6 0.6) (thickness 0.15)))
     )
-    (fp_text value 100nf (at 0 1.9 45) (layer F.Fab)
+    (fp_text value 100nf (at 0 1.9 45) (layer F.Fab) hide
       (effects (font (size 1 1) (thickness 0.15)))
     )
@@
       (xy 14 -10.3)) (layer B.SilkS) (width 0.01))
   )
+  (gr_text USB (at 143.75 78.75) (layer F.SilkS)
+    (effects (font (size 1.5 1.5) (thickness 0.3)))
+  )
+  (gr_text BLD_D- (at 139.5 83 90) (layer F.SilkS)
+    (effects (font (size 1.016 0.508) (thickness 0.127)))
+  )
+  (gr_text BLD_D+ (at 137 83 90) (layer F.SilkS)
+    (effects (font (size 1.016 0.508) (thickness 0.127)))
+  )
+  (gr_text HOST_D- (at 134.5 83.25 90) (layer F.SilkS)
+    (effects (font (size 1.016 0.508) (thickness 0.127)))
+  )
+  (gr_text HOST_D+ (at 131.75 83.25 90) (layer F.SilkS)
+    (effects (font (size 1.016 0.508) (thickness 0.127)))
+  )
   (gr_text B-Mask (at 188.341 42.545) (layer B.Mask)
     (effects (font (size 0.762 0.762) (thickness 0.1905)) (justify mirror))
@@
   (gr_arc (start 64 87) (end 64 92) (angle 90) (layer Edge.Cuts) (width 0.15))
   (gr_arc (start 64 46) (end 59 46) (angle 90) (layer Edge.Cuts) (width 0.15))
-  (dimension 40.64 (width 0.3) (layer B.CrtYd)
-    (gr_text "1.6000 in" (at 46.91 66.04 270) (layer B.CrtYd)
-      (effects (font (size 1.5 1.5) (thickness 0.3)))
-    )
-    (feature1 (pts (xy 55.88 86.36) (xy 45.56 86.36)))
-    (feature2 (pts (xy 55.88 45.72) (xy 45.56 45.72)))
-    (crossbar (pts (xy 48.26 45.72) (xy 48.26 86.36)))
-    (arrow1a (pts (xy 48.26 86.36) (xy 47.673579 85.233496)))
-    (arrow1b (pts (xy 48.26 86.36) (xy 48.846421 85.233496)))
-    (arrow2a (pts (xy 48.26 45.72) (xy 47.673579 46.846504)))
-    (arrow2b (pts (xy 48.26 45.72) (xy 48.846421 46.846504)))
-  )
   (gr_line (start 191 41) (end 191 92) (angle 90) (layer Edge.Cuts) (width 0.15))
-  (dimension 51 (width 0.3) (layer B.CrtYd)
-    (gr_text "51.000 mm" (at 212.35 66.5 270) (layer B.CrtYd)
-      (effects (font (size 1.5 1.5) (thickness 0.3)))
-    )
-    (feature1 (pts (xy 193 92) (xy 213.7 92)))
-    (feature2 (pts (xy 193 41) (xy 213.7 41)))
-    (crossbar (pts (xy 211 41) (xy 211 92)))
-    (arrow1a (pts (xy 211 92) (xy 210.413579 90.873496)))
-    (arrow1b (pts (xy 211 92) (xy 211.586421 90.873496)))
-    (arrow2a (pts (xy 211 41) (xy 210.413579 42.126504)))
-    (arrow2b (pts (xy 211 41) (xy 211.586421 42.126504)))
-  )
-  (dimension 132 (width 0.3) (layer B.CrtYd)
-    (gr_text "132.000 mm" (at 125 20.650001) (layer B.CrtYd)
-      (effects (font (size 1.5 1.5) (thickness 0.3)))
-    )
-    (feature1 (pts (xy 191 37) (xy 191 19.300001)))
-    (feature2 (pts (xy 59 37) (xy 59 19.300001)))
-    (crossbar (pts (xy 59 22.000001) (xy 191 22.000001)))
-    (arrow1a (pts (xy 191 22.000001) (xy 189.873496 22.586422)))
-    (arrow1b (pts (xy 191 22.000001) (xy 189.873496 21.41358)))
-    (arrow2a (pts (xy 59 22.000001) (xy 60.126504 22.586422)))
-    (arrow2b (pts (xy 59 22.000001) (xy 60.126504 21.41358)))
-  )
   (segment (start 119.0117 88.4301) (end 117.5893 88.4301) (width 0.3048) (layer B.Cu) (net 0))
   (segment (start 126.3777 71.3613) (end 126.85268 71.83628) (width 0.3048) (layer F.Cu) (net 1))

Commit message: new files
Parts:
- removed EE_LOGO: , logo:EE_LOGO(2)
- D1, D2, D3, D4, D5, D7, D8: footprint LEDs:LED-0603 -> EE:LED-0603_NEW
- SW2: footprint EE:Micro_slide_switch-spst_2mm -> EE:Micro_slide_switch-spst_2mm_new
Routing:
- net Net-(P3-Pad22): track 16.4 -> 19.5 mm
- net Net-(P3-Pad23): track 16.7 -> 19.2 mm
Other:
- board text added: "EINT2"
- board text added: "Explore LPC2148 Breakout"
- board text added: "RESET"
- board text added: "USB_BLD"

Commit message: added files with logo
Parts:
- added EE_LOGO: , logo:EE_LOGO(2), B.Cu at (168.0, 59.0)

Commit message: changed usb
Parts:
- removed EE_LOGO: , logo:EE_LOGO(2)
- CON2: footprint Connect:USB_Micro-B -> EE:USB_Micro-B_SMD
- moved CON2 2.02 mm to (185.2, 83.1), turned to 180 degrees

Commit message: final
Parts:
- added EE_LOGO: , logo:EE_LOGO(2), B.Cu at (168.0, 59.0)
